File: pcbart.kicad_pcb (KiCad board)
At the start: 2 copper layers, 159.1 x 29.1 mm, 4 parts

Commit message: Adjust logo
Parts:
- removed the G*** at (0.00, 0.00) (x4)
- added G*** (x5): LOGO, LOGO, F.Cu at (0.00, 0.00)
