File: ruler.sch (KiCad schematic (older format))
At the start: 25 parts, among them J1 USB_OTG, J2 Conn_01x01, SW1 KMR2, SW2 B3U-1000P, SW3 SW_Push, SW4 SW_Push, SW5 FSM2JSMA, SW6 6x6mm, SW7 JS202011SCQN

Commit message: Re-arrange push-button connections
Changed lines of the file:
@@
 	4025 5100 4025 5225
-Wire Wire Line
-	3925 4300 3950 4300
 Wire Wire Line
 	4025 4300 4025 4375
@@
 L switches:SW_Push SW3
 U 1 1 5AF1BC93
-P 5500 4075
-F 0 "SW3" H 5550 4175 50  0000 L CNN
-F 1 "SW_Push" H 5500 4015 50  0000 C CNN
-F 2 "smisioto.eu/kicad_libs/modules/w_switch.pretty:smd_push" H 5500 4275 50  0001 C CNN
-F 3 "" H 5500 4275 50  0001 C CNN
-	1    5500 4075
+P 3750 4300
+F 0 "SW3" H 3800 4400 50  0000 L CNN
+F 1 "SW_Push" H 3750 4240 50  0000 C CNN
+F 2 "smisioto.eu/kicad_libs/modules/w_switch.pretty:smd_push" H 3750 4500 50  0001 C CNN
+F 3 "" H 3750 4500 50  0001 C CNN
+	1    3750 4300
 	1    0    0    -1
 $EndComp
@@
 L switches:SW_Push SW2
 U 1 1 5AF1BCB7
-P 3725 4300
-F 0 "SW2" H 3775 4400 50  0000 L CNN
-F 1 "B3U-1000P" H 3725 4240 50  0000 C CNN
-F 2 "digikey/digikey-kicad-library/digikey-footprints.pretty:Switch_Tactile_SMD_B3U-1000P" H 3725 4500 50  0001 C CNN
-F 3 "" H 3725 4500 50  0001 C CNN
-	1    3725 4300
+P 5500 4075
+F 0 "SW2" H 5550 4175 50  0000 L CNN
+F 1 "B3U-1000P" H 5500 4015 50  0000 C CNN
+F 2 "digikey/digikey-kicad-library/digikey-footprints.pretty:Switch_Tactile_SMD_B3U-1000P" H 5500 4275 50  0001 C CNN
+F 3 "" H 5500 4275 50  0001 C CNN
+	1    5500 4075
 	1    0    0    -1
 $EndComp
@@
 Wire Wire Line
 	7475 4625 7475 4750
+Wire Wire Line
+	3550 4300 3525 4300
 $EndSCHEMATC

Commit message: Re-arrange and replace some switches
Parts:
- SW2: renamed from SW3; value SW_Push -> EVQPE1; footprint smisioto.eu/kicad_libs/modules/w_switch.pretty:smd_push -> KiCad/Buttons_Switches_SMD.pretty:SW_SPST_EVQPE1
- SW4: value SW_Push -> FSMCT
- SW5: renamed from SW6; value 6x6mm -> FSMLPU; footprint digikey/digikey-kicad-library/digikey-footprints.pretty:Switch_Tactile_6x6mm_Vertical_SMD -> digikey/digikey-kicad-library/digikey-footprints.pretty:Switch_4.5x4.5mm_SMD_TL3315NF160Q
- SW6: renamed from SW5; value FSM2JSMA -> FSM2JSM
- renumbered R4 to R3, R6 to R4, R8 to R5, SW2 to SW3
Changed lines of the file:
@@
 $EndComp
 $Comp
-L switches:SW_Push SW6
+L switches:SW_Push SW5
 U 1 1 5AF1AB0F
-P 8950 4400
-F 0 "SW6" H 8725 4600 50  0000 L CNN
-F 1 "6x6mm" H 8950 4340 50  0000 C CNN
-F 2 "digikey/digikey-kicad-library/digikey-footprints.pretty:Switch_Tactile_6x6mm_Vertical_SMD" H 8950 4600 50  0001 C CNN
-F 3 "" H 8950 4600 50  0001 C CNN
-	1    8950 4400
+P 5500 4325
+F 0 "SW5" H 5275 4525 50  0000 L CNN
+F 1 "FSMLPU" H 5500 4265 50  0000 C CNN
+F 2 "digikey/digikey-kicad-library/digikey-footprints.pretty:Switch_4.5x4.5mm_SMD_TL3315NF160Q" H 5500 4525 50  0001 C CNN
+F 3 "" H 5500 4525 50  0001 C CNN
+	1    5500 4325
 	1    0    0    -1
 $EndComp
@@
 L switches:SW_Push SW4
 U 1 1 5AF1B6F7
-P 5500 4325
-F 0 "SW4" H 5550 4425 50  0000 L CNN
-F 1 "SW_Push" H 5500 4265 50  0000 C CNN
-F 2 "smisioto.eu/kicad_libs/modules/w_switch.pretty:smd_push2" H 5500 4525 50  0001 C CNN
-F 3 "" H 5500 4525 50  0001 C CNN
-	1    5500 4325
-	1    0    0    -1
-$EndComp
-$Comp
-L device:R R4
+P 7175 4250
+F 0 "SW4" H 7225 4350 50  0000 L CNN
+F 1 "FSMCT" H 7175 4190 50  0000 C CNN
+F 2 "smisioto.eu/kicad_libs/modules/w_switch.pretty:smd_push2" H 7175 4450 50  0001 C CNN
+F 3 "" H 7175 4450 50  0001 C CNN
+	1    7175 4250
+	1    0    0    -1
+$EndComp
+$Comp
+L device:R R3
 U 1 1 5AF1B6FD
 P 5900 4550
-F 0 "R4" V 5980 4550 50  0000 C CNN
+F 0 "R3" V 5980 4550 50  0000 C CNN
 F 1 "1k" V 5900 4550 50  0000 C CNN
 F 2 "KiCad/Resistors_SMD.pretty:R_0603" V 5830 4550 50  0001 C CNN
@@
 	5900 4325 5900 4400
 $Comp
-L switches:SW_Push SW3
+L switches:SW_Push SW2
 U 1 1 5AF1BC93
 P 3750 4300
-F 0 "SW3" H 3800 4400 50  0000 L CNN
-F 1 "SW_Push" H 3750 4240 50  0000 C CNN
-F 2 "smisioto.eu/kicad_libs/modules/w_switch.pretty:smd_push" H 3750 4500 50  0001 C CNN
+F 0 "SW2" H 3800 4400 50  0000 L CNN
+F 1 "EVQPE1" H 3750 4240 50  0000 C CNN
+F 2 "KiCad/Buttons_Switches_SMD.pretty:SW_SPST_EVQPE1" H 3750 4500 50  0001 C CNN
 F 3 "" H 3750 4500 50  0001 C CNN
 	1    3750 4300
@@
 $EndComp
 $Comp
-L device:R R6
+L device:R R4
 U 1 1 5AF1BC99
 P 7475 4475
-F 0 "R6" V 7555 4475 50  0000 C CNN
+F 0 "R4" V 7555 4475 50  0000 C CNN
 F 1 "1k" V 7475 4475 50  0000 C CNN
 F 2 "KiCad/Resistors_SMD.pretty:R_0805" V 7405 4475 50  0001 C CNN
@@
 	7475 4250 7475 4325
 $Comp
-L switches:SW_Push SW2
+L switches:SW_Push SW3
 U 1 1 5AF1BCB7
 P 5500 4075
-F 0 "SW2" H 5550 4175 50  0000 L CNN
+F 0 "SW3" H 5550 4175 50  0000 L CNN
 F 1 "B3U-1000P" H 5500 4015 50  0000 C CNN
 F 2 "digikey/digikey-kicad-library/digikey-footprints.pretty:Switch_Tactile_SMD_B3U-1000P" H 5500 4275 50  0001 C CNN
@@
 $EndComp
 $Comp
-L device:R R8
+L device:R R5
 U 1 1 5AF1BCBD
 P 9250 4625
-F 0 "R8" V 9330 4625 50  0000 C CNN
+F 0 "R5" V 9330 4625 50  0000 C CNN
 F 1 "1k" V 9250 4625 50  0000 C CNN
 F 2 "KiCad/Resistors_SMD.pretty:R_1206" V 9180 4625 50  0001 C CNN
@@
 	3475 4300 3525 4300
 $Comp
-L switches:SW_Push SW5
+L switches:SW_Push SW6
 U 1 1 5AF214E5
-P 7175 4250
-F 0 "SW5" H 6950 4450 50  0000 L CNN
-F 1 "FSM2JSMA" H 7175 4190 50  0000 C CNN
-F 2 "custom:FSM2JSMA" H 7175 4450 50  0001 C CNN
-F 3 "" H 7175 4450 50  0001 C CNN
-	1    7175 4250
-	1    0    0    -1
-$EndComp
+P 8950 4400
+F 0 "SW6" H 8725 4600 50  0000 L CNN
+F 1 "FSM2JSM" H 8950 4340 50  0000 C CNN
+F 2 "custom:FSM2JSMA" H 8950 4600 50  0001 C CNN
+F 3 "" H 8950 4600 50  0001 C CNN
+	1    8950 4400
+	1    0    0    -1
+$EndComp

Commit message: Adjust led test pads
Parts:
- SW3: value B3U-1000P -> B3U1000P
Changed lines of the file:
@@
 U 1 1 5AF1AB0F
 P 5500 4325
-F 0 "SW5" H 5275 4525 50  0000 L CNN
+F 0 "SW5" H 5575 4400 50  0000 L CNN
 F 1 "FSMLPU" H 5500 4265 50  0000 C CNN
 F 2 "digikey/digikey-kicad-library/digikey-footprints.pretty:Switch_4.5x4.5mm_SMD_TL3315NF160Q" H 5500 4525 50  0001 C CNN
@@
 P 5500 4075
 F 0 "SW3" H 5550 4175 50  0000 L CNN
-F 1 "B3U-1000P" H 5500 4015 50  0000 C CNN
+F 1 "B3U1000P" H 5500 4015 50  0000 C CNN
 F 2 "digikey/digikey-kicad-library/digikey-footprints.pretty:Switch_Tactile_SMD_B3U-1000P" H 5500 4275 50  0001 C CNN
 F 3 "" H 5500 4275 50  0001 C CNN

Commit message: Route route route
Parts:
- SW4: footprint smisioto.eu/kicad_libs/modules/w_switch.pretty:smd_push2 -> custom:FSMCT; symbol switches:SW_Push -> switches:SW_Push_Dual
- SW5: value FSMLPU -> TL3315; symbol switches:SW_Push -> switches:SW_Push_Dual
Connections:
- wire segments 62 -> 78
Changed lines of the file:
@@
-$EndComp
-$Comp
-L switches:SW_Push SW5
-U 1 1 5AF1AB0F
-P 5500 4325
-F 0 "SW5" H 5575 4400 50  0000 L CNN
-F 1 "FSMLPU" H 5500 4265 50  0000 C CNN
-F 2 "digikey/digikey-kicad-library/digikey-footprints.pretty:Switch_4.5x4.5mm_SMD_TL3315NF160Q" H 5500 4525 50  0001 C CNN
-F 3 "" H 5500 4525 50  0001 C CNN
-	1    5500 4325
-	1    0    0    -1
 $EndComp
 $Comp
@@
 Connection ~ 900  3050
 $Comp
-L switches:SW_Push SW4
+L switches:SW_Push_Dual SW4
 U 1 1 5AF1B6F7
-P 7175 4250
-F 0 "SW4" H 7225 4350 50  0000 L CNN
-F 1 "FSMCT" H 7175 4190 50  0000 C CNN
-F 2 "smisioto.eu/kicad_libs/modules/w_switch.pretty:smd_push2" H 7175 4450 50  0001 C CNN
-F 3 "" H 7175 4450 50  0001 C CNN
-	1    7175 4250
-	1    0    0    -1
+P 7250 4775
+F 0 "SW4" H 7300 4875 50  0000 L CNN
+F 1 "FSMCT" H 7250 4715 50  0000 C CNN
+F 2 "custom:FSMCT" H 7250 4975 50  0001 C CNN
+F 3 "" H 7250 4975 50  0001 C CNN
+	1    7250 4775
+	0    1    1    0
 $EndComp
 $Comp
@@
 	5900 5125 5900 5250
 Wire Wire Line
-	4975 4325 5300 4325
-Wire Wire Line
-	5700 4325 5775 4325
-Wire Wire Line
 	5900 4325 5900 4400
 $Comp
@@
 	6825 4100 6825 4250
 Wire Wire Line
-	6825 4250 6975 4250
-Wire Wire Line
-	7375 4250 7475 4250
-Wire Wire Line
 	7475 4250 7475 4325
 $Comp
@@
 	9250 5200 9250 5325
 Wire Wire Line
-	8575 4400 8750 4400
-Wire Wire Line
-	9150 4400 9250 4400
-Wire Wire Line
 	9250 4400 9250 4475
 Wire Wire Line
@@
 	3475 4300 3525 4300
 $Comp
+L switches:SW_Push SW1
+U 1 1 5AF21638
+P 3725 3950
+F 0 "SW1" H 3500 4150 50  0000 L CNN
+F 1 "KMR2" H 3725 3890 50  0000 C CNN
+F 2 "KiCad/Buttons_Switches_SMD.pretty:SW_SPST_KMR2" H 3725 4150 50  0001 C CNN
+F 3 "" H 3725 4150 50  0001 C CNN
+	1    3725 3950
+	1    0    0    -1
+$EndComp
+Wire Wire Line
+	5300 4075 4975 4075
+Wire Wire Line
+	4975 4075 4975 4175
+Wire Wire Line
+	4925 4175 4975 4175
+Connection ~ 4975 4175
+Wire Wire Line
+	4975 4175 4975 4325
+Wire Wire Line
+	5700 4075 5775 4075
+Wire Wire Line
+	5775 4075 5775 4325
+Connection ~ 5775 4325
+Wire Wire Line
+	5775 4325 5900 4325
+Text GLabel 4175 3775 1    50   Input ~ 0
+LED_V+
+Wire Wire Line
+	3525 3950 3525 4300
+Connection ~ 3525 4300
+Wire Wire Line
+	3950 4300 3950 3950
+Wire Wire Line
+	3950 3950 3925 3950
+Connection ~ 3950 4300
+Wire Wire Line
+	3950 4300 4025 4300
+$Comp
+L device:D D1
+U 1 1 5AF423A2
+P 6050 4150
+F 0 "D1" V 6096 4071 50  0000 R CNN
+F 1 "SMA" V 6005 4071 50  0000 R CNN
+F 2 "KiCad/Diodes_SMD.pretty:D_SMA" H 6050 4150 50  0001 C CNN
+F 3 "" H 6050 4150 50  0001 C CNN
+	1    6050 4150
+	0    -1   -1   0
+$EndComp
+Wire Wire Line
+	4175 3775 4175 3975
+Wire Wire Line
+	4175 4275 4175 4300
+Wire Wire Line
+	4175 4300 4025 4300
+Connection ~ 4025 4300
+Wire Wire Line
+	4025 4675 4025 4800
+Wire Wire Line
+	5900 4700 5900 4825
+Text GLabel 6050 3800 1    50   Input ~ 0
+LED_V+
+$Comp
+L device:D D2
+U 1 1 5AF48CEA
+P 9400 4225
+F 0 "D2" V 9446 4146 50  0000 R CNN
+F 1 "SMB" V 9355 4146 50  0000 R CNN
+F 2 "KiCad/Diodes_SMD.pretty:D_SMB" H 9400 4225 50  0001 C CNN
+F 3 "" H 9400 4225 50  0001 C CNN
+	1    9400 4225
+	0    -1   -1   0
+$EndComp
+Wire Wire Line
+	6050 3800 6050 4000
+Wire Wire Line
+	6050 4300 6050 4325
+Wire Wire Line
+	6050 4325 5900 4325
+Connection ~ 5900 4325
+Text GLabel 7625 3725 1    50   Input ~ 0
+LED_V+
+$Comp
+L device:D D3
+U 1 1 5AF49F44
+P 4175 4125
+F 0 "D3" V 4221 4046 50  0000 R CNN
+F 1 "SMC" V 4130 4046 50  0000 R CNN
+F 2 "KiCad/Diodes_SMD.pretty:D_SMC" H 4175 4125 50  0001 C CNN
+F 3 "" H 4175 4125 50  0001 C CNN
+	1    4175 4125
+	0    -1   -1   0
+$EndComp
+Wire Wire Line
+	7625 3725 7625 3925
+Wire Wire Line
+	7625 4225 7625 4250
+Wire Wire Line
+	7625 4250 7475 4250
+Connection ~ 7475 4250
+Text GLabel 9400 3875 1    50   Input ~ 0
+LED_V+
+$Comp
+L device:D D4
+U 1 1 5AF4B2D9
+P 7625 4075
+F 0 "D4" V 7671 3996 50  0000 R CNN
+F 1 "SOD-123" V 7580 3996 50  0000 R CNN
+F 2 "KiCad/Diodes_SMD.pretty:D_SOD-123" H 7625 4075 50  0001 C CNN
+F 3 "" H 7625 4075 50  0001 C CNN
+	1    7625 4075
+	0    -1   -1   0
+$EndComp
+Wire Wire Line
+	9400 3875 9400 4075
+Wire Wire Line
+	9400 4375 9400 4400
+Wire Wire Line
+	9400 4400 9250 4400
+Connection ~ 9250 4400
+Wire Wire Line
+	9250 4775 9250 4900
+$Comp
+L device:D D5
+U 1 1 5AF4E276
+P 9950 4225
+F 0 "D5" V 9996 4146 50  0000 R CNN
+F 1 "SOD-323" V 9905 4146 50  0000 R CNN
+F 2 "KiCad/Diodes_SMD.pretty:D_SOD-323" H 9950 4225 50  0001 C CNN
+F 3 "" H 9950 4225 50  0001 C CNN
+	1    9950 4225
+	0    -1   -1   0
+$EndComp
+$Comp
+L device:D D6
+U 1 1 5AF4E2E0
+P 10550 4200
+F 0 "D6" V 10596 4121 50  0000 R CNN
+F 1 "SOD-523" V 10505 4121 50  0000 R CNN
+F 2 "KiCad/Diodes_SMD.pretty:D_SOD-523" H 10550 4200 50  0001 C CNN
+F 3 "" H 10550 4200 50  0001 C CNN
+	1    10550 4200
+	0    -1   -1   0
+$EndComp
+Wire Wire Line
+	3550 4300 3525 4300
+$Comp
 L switches:SW_Push SW6
 U 1 1 5AF214E5
@@
 	1    0    0    -1
 $EndComp
-$Comp
-L switches:SW_Push SW1
-U 1 1 5AF21638
-P 3725 3950
-F 0 "SW1" H 3500 4150 50  0000 L CNN
-F 1 "KMR2" H 3725 3890 50  0000 C CNN
-F 2 "KiCad/Buttons_Switches_SMD.pretty:SW_SPST_KMR2" H 3725 4150 50  0001 C CNN
-F 3 "" H 3725 4150 50  0001 C CNN
-	1    3725 3950
-	1    0    0    -1
-$EndComp
-Wire Wire Line
-	5300 4075 4975 4075
-Wire Wire Line
-	4975 4075 4975 4175
-Wire Wire Line
-	4925 4175 4975 4175
-Connection ~ 4975 4175
-Wire Wire Line
-	4975 4175 4975 4325
-Wire Wire Line
-	5700 4075 5775 4075
-Wire Wire Line
-	5775 4075 5775 4325
-Connection ~ 5775 4325
-Wire Wire Line
-	5775 4325 5900 4325
-Text GLabel 4175 3775 1    50   Input ~ 0
-LED_V+
-Wire Wire Line
-	3525 3950 3525 4300
-Connection ~ 3525 4300
-Wire Wire Line
-	3950 4300 3950 3950
-Wire Wire Line
-	3950 3950 3925 3950
-Connection ~ 3950 4300
-Wire Wire Line
-	3950 4300 4025 4300
-$Comp
-L device:D D1
-U 1 1 5AF423A2
-P 4175 4125
-F 0 "D1" V 4221 4046 50  0000 R CNN
-F 1 "SMA" V 4130 4046 50  0000 R CNN
-F 2 "KiCad/Diodes_SMD.pretty:D_SMA" H 4175 4125 50  0001 C CNN
-F 3 "" H 4175 4125 50  0001 C CNN
-	1    4175 4125
-	0    -1   -1   0
-$EndComp
-Wire Wire Line
-	4175 3775 4175 3975
-Wire Wire Line
-	4175 4275 4175 4300
-Wire Wire Line
-	4175 4300 4025 4300
-Connection ~ 4025 4300
-Wire Wire Line
-	4025 4675 4025 4800
-Wire Wire Line
-	5900 4700 5900 4825
-Text GLabel 6050 3800 1    50   Input ~ 0
-LED_V+
-$Comp
-L device:D D2
-U 1 1 5AF48CEA
-P 6050 4150
-F 0 "D2" V 6096 4071 50  0000 R CNN
-F 1 "SMB" V 6005 4071 50  0000 R CNN
-F 2 "KiCad/Diodes_SMD.pretty:D_SMB" H 6050 4150 50  0001 C CNN
-F 3 "" H 6050 4150 50  0001 C CNN
-	1    6050 4150
-	0    -1   -1   0
-$EndComp
-Wire Wire Line
-	6050 3800 6050 4000
-Wire Wire Line
-	6050 4300 6050 4325
-Wire Wire Line
-	6050 4325 5900 4325
-Connection ~ 5900 4325
-Text GLabel 7625 3725 1    50   Input ~ 0
-LED_V+
-$Comp
-L device:D D3
-U 1 1 5AF49F44
-P 7625 4075
-F 0 "D3" V 7671 3996 50  0000 R CNN
-F 1 "SMC" V 7580 3996 50  0000 R CNN
-F 2 "KiCad/Diodes_SMD.pretty:D_SMC" H 7625 4075 50  0001 C CNN
-F 3 "" H 7625 4075 50  0001 C CNN
-	1    7625 4075
-	0    -1   -1   0
-$EndComp
-Wire Wire Line
-	7625 3725 7625 3925
-Wire Wire Line
-	7625 4225 7625 4250
-Wire Wire Line
-	7625 4250 7475 4250
-Connection ~ 7475 4250
-Text GLabel 9400 3875 1    50   Input ~ 0
-LED_V+
-$Comp
-L device:D D4
-U 1 1 5AF4B2D9
-P 9400 4225
-F 0 "D4" V 9446 4146 50  0000 R CNN
-F 1 "SOD-123" V 9355 4146 50  0000 R CNN
-F 2 "KiCad/Diodes_SMD.pretty:D_SOD-123" H 9400 4225 50  0001 C CNN
-F 3 "" H 9400 4225 50  0001 C CNN
-	1    9400 4225
-	0    -1   -1   0
-$EndComp
-Wire Wire Line
-	9400 3875 9400 4075
-Wire Wire Line
-	9400 4375 9400 4400
-Wire Wire Line
-	9400 4400 9250 4400
-Connection ~ 9250 4400
-Wire Wire Line
-	9250 4775 9250 4900
-$Comp
-L device:D D5
-U 1 1 5AF4E276
-P 9950 4225
-F 0 "D5" V 9996 4146 50  0000 R CNN
-F 1 "SOD-323" V 9905 4146 50  0000 R CNN
-F 2 "KiCad/Diodes_SMD.pretty:D_SOD-323" H 9950 4225 50  0001 C CNN
-F 3 "" H 9950 4225 50  0001 C CNN
-	1    9950 4225
-	0    -1   -1   0
-$EndComp
-$Comp
-L device:D D6
-U 1 1 5AF4E2E0
-P 10550 4200
-F 0 "D6" V 10596 4121 50  0000 R CNN
-F 1 "SOD-523" V 10505 4121 50  0000 R CNN
-F 2 "KiCad/Diodes_SMD.pretty:D_SOD-523" H 10550 4200 50  0001 C CNN
-F 3 "" H 10550 4200 50  0001 C CNN
-	1    10550 4200
-	0    -1   -1   0
-$EndComp
+Wire Wire Line
+	9150 4400 9250 4400
+Wire Wire Line
+	8575 4400 8750 4400
+$Comp
+L switches:SW_Push_Dual SW5
+U 1 1 5AF1AB0F
+P 5575 4600
+F 0 "SW5" H 5650 4675 50  0000 L CNN
+F 1 "TL3315" H 5575 4540 50  0000 C CNN
+F 2 "digikey/digikey-kicad-library/digikey-footprints.pretty:Switch_4.5x4.5mm_SMD_TL3315NF160Q" H 5575 4800 50  0001 C CNN
+F 3 "" H 5575 4800 50  0001 C CNN
+	1    5575 4600
+	0    1    1    0
+$EndComp
+Wire Wire Line
+	4975 4325 5375 4325
+Wire Wire Line
+	5575 4325 5775 4325
+Wire Wire Line
+	5375 4325 5375 4400
+Connection ~ 5375 4400
+Wire Wire Line
+	5375 4400 5375 4800
+Wire Wire Line
+	5575 4325 5575 4400
+Connection ~ 5575 4400
+Wire Wire Line
+	5575 4400 5575 4800
+Wire Wire Line
+	6825 4250 7075 4250
+Wire Wire Line
+	7275 4250 7475 4250
+Wire Wire Line
+	7075 4250 7075 4325
+Wire Wire Line
+	7275 4250 7275 4325
+Wire Wire Line
+	7075 4325 6950 4325
+Wire Wire Line
+	6950 4325 6950 4525
 Wire Wire Line
 	7475 4625 7475 4750
 Wire Wire Line
-	3550 4300 3525 4300
+	7275 4325 7350 4325
+Wire Wire Line
+	7350 4325 7350 4525
+Wire Wire Line
+	7050 4575 7050 4975
+Wire Wire Line
+	7250 4575 7250 4975
+Wire Wire Line
+	6950 4525 7050 4525
+Wire Wire Line
+	7050 4525 7050 4575
+Connection ~ 7050 4575
+Wire Wire Line
+	7250 4575 7250 4525
+Wire Wire Line
+	7250 4525 7350 4525
+Connection ~ 7250 4575
 $EndSCHEMATC

Commit message: Add inductors, caps, transitors and ICs
Parts:
- added C1: 3x5.3mm, KiCad/Capacitors_SMD.pretty:CP_Elec_3x5.3, symbol device:CP
- added C2: 4x5.8mm, KiCad/Capacitors_SMD.pretty:CP_Elec_4x5.8, symbol device:CP
- added C3: 5x5.8mm, KiCad/Capacitors_SMD.pretty:CP_Elec_5x5.8, symbol device:CP
- added C4: 8x5.4mm, KiCad/Capacitors_SMD.pretty:CP_Elec_8x5.4, symbol device:CP
- added C5: A/3216, KiCad/Capacitors_Tantalum_SMD.pretty:CP_Tantalum_Case-A_EIA-3216-18_Reflow, symbol device:CP
- added C6: B/3528, KiCad/Capacitors_Tantalum_SMD.pretty:CP_Tantalum_Case-B_EIA-3528-21_Reflow, symbol device:CP
- added C7: C/6032, KiCad/Capacitors_Tantalum_SMD.pretty:CP_Tantalum_Case-C_EIA-6032-28_Reflow, symbol device:CP
- added C8: D/7343, KiCad/Capacitors_Tantalum_SMD.pretty:CP_Tantalum_Case-D_EIA-7343-31_Reflow, symbol device:CP
- added L1: 1008, jnedbal/jakub.pretty:Inductor_1008, symbol pspice:INDUCTOR
- added L2: SRU8043, custom:Inductor_Bourns-SRU8043, symbol pspice:INDUCTOR
- added L3: 4040, KiCad/Inductors.pretty:Inductor_Taiyo-Yuden_MD-4040, symbol pspice:INDUCTOR
- added L4: 5050, KiCad/Inductors.pretty:Inductor_Taiyo-Yuden_MD-5050, symbol pspice:INDUCTOR
- added L5: 60xx, KiCad/Inductors.pretty:Inductor_Taiyo-Yuden_NR-60xx, symbol pspice:INDUCTOR
- added Q1: Q_NMOS_DGS, adamgreig/agg-kicad/agg.pretty:SOT-23, symbol device:Q_NMOS_DGS
- added Q2: Q_NMOS_DGS, adamgreig/agg-kicad/agg.pretty:SOT-323, symbol device:Q_NMOS_DGS
- added Q3: Q_NMOS_DGS, adamgreig/agg-kicad/agg.pretty:SOT-883-B, symbol device:Q_NMOS_DGS
- added Q4: Q_NMOS_DGS, digikey/digikey-kicad-library/digikey-footprints.pretty:SOT-523, symbol device:Q_NMOS_DGS
- added Q5: Q_NMOS_DGS, ep092/library_toni.pretty:SOT223_GND_VO_VI, symbol device:Q_NMOS_DGS
- added U1: Conn_01x01, KiCad/Housings_DFN_QFN.pretty:QFN-16-1EP_3x3mm_Pitch0.5mm, symbol conn:Conn_01x01
- added U2: Conn_01x01, adamgreig/agg-kicad/agg.pretty:LQFP-32, symbol conn:Conn_01x01
- added U3: Conn_01x01, adamgreig/agg-kicad/agg.pretty:SOIC-8, symbol conn:Conn_01x01
- added U4: Conn_01x01, KiCad/SMD_Packages.pretty:BGA-64-0.8mm, symbol conn:Conn_01x01
- added U5: Conn_01x01, KiCad/Housings_SSOP.pretty:TSSOP-16_4.4x5mm_Pitch0.65mm, symbol conn:Conn_01x01
- renumbered J2 to DRAWING1

Commit message: Change text to inkscape versions
Parts:
- DRAWING1: footprint drawing:drawing -> drawings:ruler
Changed lines of the file:
@@
 F 0 "DRAWING1" H 10925 6300 50  0000 C CNN
 F 1 "Conn_01x01" H 10925 6100 50  0000 C CNN
-F 2 "drawing:drawing" H 10925 6200 50  0001 C CNN
+F 2 "drawings:ruler" H 10925 6200 50  0001 C CNN
 F 3 "" H 10925 6200 50  0001 C CNN
 	1    10925 6200

Commit message: Adjust title texts
Parts:
- added DRAWING2: Conn_01x01, drawings:leds_text, symbol conn:Conn_01x01
- added DRAWING3: Conn_01x01, drawings:resistors_text, symbol conn:Conn_01x01
- added DRAWING4: Conn_01x01, drawings:diodes_text, symbol conn:Conn_01x01
- added DRAWING5: Conn_01x01, drawings:switches_text, symbol conn:Conn_01x01
Changed lines of the file:
@@
+	1    0    0    -1
+$EndComp
+$Comp
+L conn:Conn_01x01 DRAWING2
+U 1 1 5AF38CEB
+P 10850 5800
+F 0 "DRAWING2" H 10850 5900 50  0000 C CNN
+F 1 "Conn_01x01" H 10850 5700 50  0000 C CNN
+F 2 "drawings:leds_text" H 10850 5800 50  0001 C CNN
+F 3 "" H 10850 5800 50  0001 C CNN
+	1    10850 5800
+	1    0    0    -1
+$EndComp
+$Comp
+L conn:Conn_01x01 DRAWING3
+U 1 1 5AF3917C
+P 10200 5825
+F 0 "DRAWING3" H 10200 5925 50  0000 C CNN
+F 1 "Conn_01x01" H 10200 5725 50  0000 C CNN
+F 2 "drawings:resistors_text" H 10200 5825 50  0001 C CNN
+F 3 "" H 10200 5825 50  0001 C CNN
+	1    10200 5825
+	1    0    0    -1
+$EndComp
+$Comp
+L conn:Conn_01x01 DRAWING4
+U 1 1 5AF3941C
+P 10150 6200
+F 0 "DRAWING4" H 10150 6300 50  0000 C CNN
+F 1 "Conn_01x01" H 10150 6100 50  0000 C CNN
+F 2 "drawings:diodes_text" H 10150 6200 50  0001 C CNN
+F 3 "" H 10150 6200 50  0001 C CNN
+	1    10150 6200
+	1    0    0    -1
+$EndComp
+$Comp
+L conn:Conn_01x01 DRAWING5
+U 1 1 5AF39890
+P 9700 5800
+F 0 "DRAWING5" H 9700 5900 50  0000 C CNN
+F 1 "Conn_01x01" H 9700 5700 50  0000 C CNN
+F 2 "drawings:switches_text" H 9700 5800 50  0001 C CNN
+F 3 "" H 9700 5800 50  0001 C CNN
+	1    9700 5800
 	1    0    0    -1
 $EndComp

Commit message: Adjust led tester text
Parts:
- added DRAWING10: Conn_01x01, drawings:tantalum_text, symbol conn:Conn_01x01
- added DRAWING11: Conn_01x01, drawings:electrolytic_text, symbol conn:Conn_01x01
- added DRAWING12: Conn_01x01, drawings:vscore, symbol conn:Conn_01x01
- added DRAWING6: Conn_01x01, drawings:capacitors_text, symbol conn:Conn_01x01
- added DRAWING7: Conn_01x01, drawings:transistors_text, symbol conn:Conn_01x01
- added DRAWING8: Conn_01x01, drawings:ics_text, symbol conn:Conn_01x01
- added DRAWING9: Conn_01x01, drawings:inductors_text, symbol conn:Conn_01x01
- LED1: value LED TEST PADS -> LED Tester
Changed lines of the file:
@@
 P 2275 1825
 F 0 "LED1" H 2275 1925 50  0000 C CNN
-F 1 "LED TEST PADS" H 2275 1725 50  0000 C CNN
+F 1 "LED Tester" H 2275 1725 50  0000 C CNN
 F 2 "custom:led_test_pads" H 2275 1825 50  0001 C CNN
 F 3 "" H 2275 1825 50  0001 C CNN
@@
 	1    0    0    -1
 $EndComp
+$Comp
+L conn:Conn_01x01 DRAWING6
+U 1 1 5AF3813A
+P 9650 6200
+F 0 "DRAWING6" H 9650 6300 50  0000 C CNN
+F 1 "Conn_01x01" H 9650 6100 50  0000 C CNN
+F 2 "drawings:capacitors_text" H 9650 6200 50  0001 C CNN
+F 3 "" H 9650 6200 50  0001 C CNN
+	1    9650 6200
+	1    0    0    -1
+$EndComp
+$Comp
+L conn:Conn_01x01 DRAWING9
+U 1 1 5AF38772
+P 9075 6200
+F 0 "DRAWING9" H 9075 6300 50  0000 C CNN
+F 1 "Conn_01x01" H 9075 6100 50  0000 C CNN
+F 2 "drawings:inductors_text" H 9075 6200 50  0001 C CNN
+F 3 "" H 9075 6200 50  0001 C CNN
+	1    9075 6200
+	1    0    0    -1
+$EndComp
+$Comp
+L conn:Conn_01x01 DRAWING8
+U 1 1 5AF388C7
+P 8575 6150
+F 0 "DRAWING8" H 8575 6250 50  0000 C CNN
+F 1 "Conn_01x01" H 8575 6050 50  0000 C CNN
+F 2 "drawings:ics_text" H 8575 6150 50  0001 C CNN
+F 3 "" H 8575 6150 50  0001 C CNN
+	1    8575 6150
+	1    0    0    -1
+$EndComp
+$Comp
+L conn:Conn_01x01 DRAWING7
+U 1 1 5AF38B4D
+P 8125 6150
+F 0 "DRAWING7" H 8125 6250 50  0000 C CNN
+F 1 "Conn_01x01" H 8125 6050 50  0000 C CNN
+F 2 "drawings:transistors_text" H 8125 6150 50  0001 C CNN
+F 3 "" H 8125 6150 50  0001 C CNN
+	1    8125 6150
+	1    0    0    -1
+$EndComp
+$Comp
+L conn:Conn_01x01 DRAWING11
+U 1 1 5AF39663
+P 8250 5750
+F 0 "DRAWING11" H 8250 5850 50  0000 C CNN
+F 1 "Conn_01x01" H 8250 5650 50  0000 C CNN
+F 2 "drawings:electrolytic_text" H 8250 5750 50  0001 C CNN
+F 3 "" H 8250 5750 50  0001 C CNN
+	1    8250 5750
+	1    0    0    -1
+$EndComp
+$Comp
+L conn:Conn_01x01 DRAWING10
+U 1 1 5AF39963
+P 7725 5800
+F 0 "DRAWING10" H 7725 5900 50  0000 C CNN
+F 1 "Conn_01x01" H 7725 5700 50  0000 C CNN
+F 2 "drawings:tantalum_text" H 7725 5800 50  0001 C CNN
+F 3 "" H 7725 5800 50  0001 C CNN
+	1    7725 5800
+	1    0    0    -1
+$EndComp
+$Comp
+L conn:Conn_01x01 DRAWING12
+U 1 1 5AF3A08D
+P 7675 6225
+F 0 "DRAWING12" H 7675 6325 50  0000 C CNN
+F 1 "Conn_01x01" H 7675 6125 50  0000 C CNN
+F 2 "drawings:vscore" H 7675 6225 50  0001 C CNN
+F 3 "" H 7675 6225 50  0001 C CNN
+	1    7675 6225
+	1    0    0    -1
+$EndComp
